Commit message: add navigation

File: iqr_4b_description/urdf/iqr_4b_robot.urdf.xacro (robot description, xacro)
@@ -32,4 +32,4 @@
   </xacro:kinect_v2>
   <!-- Kinova jaco j2n6s300 -->
-  <xacro:j2n6s300  base_parent="arm_mount_link"/>
+  <!--xacro:j2n6s300  base_parent="arm_mount_link"/-->
 </robot>

File: iqr_4b_description/urdf/vlp16.xacro (robot description, xacro)
@@ -19,9 +19,9 @@
       <child link="${prefix}_link"/>
     </joint>
-    <link name="laser"/>
-    <joint name="laser_link_joint" type="fixed">
+    <link name="velodyne"/>
+    <joint name="velodyne_link_joint" type="fixed">
       <origin xyz="0 0 0.040" rpy="0 0 0" />
       <parent link="${prefix}_link"/>
-      <child link="laser"/>
+      <child link="velodyne"/>
     </joint>
   </xacro:macro>
